Commit message: change: Updated controller parameters and the wist2_joint limits

File: src/robotics_project/urdf/arm_assembly.urdf (robot description, URDF)
Before this commit: robot arm_assembly, 11 links, 10 joints
Joints:
- joint wrist_1_joint: limit lower=0 upper=3.14 effort=100.0 velocity=3.0 -> lower=-1.57 upper=1.57 effort=100.0 velocity=3.0

Commit message: updated .gitignore and edited sedf and pose_executor.py and yamlfile

File: src/robotics_project/urdf/arm_assembly.urdf (robot description, URDF)
Before this commit: robot arm_assembly, 11 links, 10 joints
Joints:
- joint shoulder_joint: limit lower=0 upper=3.14 effort=100.0 velocity=3.0 -> lower=-0.01 upper=3.14 effort=100.0 velocity=3.0
